File: fanpcb/fanpcb.kicad_pcb (KiCad board)
At the start: 2 copper layers, 30 x 50 mm, 16 parts, among them M1 Fan_4pin, M2 Fan_4pin, M3 Fan_4pin, T1 TACHO, T12V1 TestPoint, T2 TACHO, T3 TACHO

Commit message: Mounting Holes added, gerber updated
Parts:
- added H1: MountingHole_Pad, MountingHole:MountingHole_3.2mm_M3_DIN965_Pad_TopBottom, F.Cu at (108.0, 115.0)
- added H2: MountingHole_Pad, MountingHole:MountingHole_3.2mm_M3_DIN965_Pad_TopBottom, F.Cu at (108.1, 126.1)
